File: LFR_MCB/LFR_MCB.kicad_pcb (KiCad board)
At the start: 2 copper layers, 81 x 81.5 mm, 17 parts, among them J1 Screw_Terminal_01x02, J10 Conn_01x08_Socket, J2 Screw_Terminal_01x02, J3 Screw_Terminal_01x02, J4 Conn_01x15_Socket, J5 Conn_01x15_Socket, J6 Conn_01x15_Socket, J9 Conn_01x08_Socket, SW1 SW_Wuerth_450301014042, SW2 SW_Push, SW3 SW_Push, U1 LM2931AZ-5.0_TO92

Commit message: Add ngspice configuration and update schematic with new junctions and wires
- Introduced ngspice settings in the project configuration file to enhance simulation capabilities.
- Added a new junction at coordinates (92.71, 72.39) in the schematic.
- Removed an unnecessary no_connect element and replaced it with a wire connecting the new junction.
- Updated UUIDs for multiple pins to ensure uniqueness across the schematic.
- Created a lock file to manage project access and prevent concurrent modifications.
Connections:
- C1 pad 2: Net-(J5-Pin_15) -> Net-(J4-Pin_15)
- J4 pad 15: unconnected-(J4-Pin_15-Pad15) -> Net-(J4-Pin_15)
- J5 pad 15: Net-(J5-Pin_15) -> Net-(J4-Pin_15)
- J9 pad 2: Net-(J5-Pin_15) -> Net-(J4-Pin_15)
- U1 pad 1: Net-(J5-Pin_15) -> Net-(J4-Pin_15)
Routing:
- net Net-(J4-Pin_15): track 0.00 -> 79.8 mm
- net Net-(J5-Pin_15): track 75.2 -> 0.00 mm
