File: LFR_MCB/LFR_MCB.kicad_sch (KiCad schematic)
At the start: 17 parts, among them J1 Screw_Terminal_01x02, J10 Conn_01x08_Socket, J2 Screw_Terminal_01x02, J3 Screw_Terminal_01x02, J4 Conn_01x15_Socket, J5 Conn_01x15_Socket, J6 Conn_01x15_Socket, J9 Conn_01x08_Socket, SW1 SW_Wuerth_450301014042, SW2 SW_Push, SW3 SW_Push, U1 LM2931AZ-5.0_TO92

Commit message: Add ngspice configuration and update schematic with new junctions and wires
- Introduced ngspice settings in the project configuration file to enhance simulation capabilities.
- Added a new junction at coordinates (92.71, 72.39) in the schematic.
- Removed an unnecessary no_connect element and replaced it with a wire connecting the new junction.
- Updated UUIDs for multiple pins to ensure uniqueness across the schematic.
- Created a lock file to manage project access and prevent concurrent modifications.
Connections:
- net at C1.2, J5.15 (Pin_15), J9.2 (Pin_2)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: now also J4.15 (Pin_15)
- no-connect marks 16 -> 15
Changed lines of the file:
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@@
+	)
+	(junction
+		(at 92.71 72.39)
+		(diameter 0)
+		(color 0 0 0 0)
 	)
 	(junction
@@
 	)
 	(no_connect
-		(at 74.93 72.39)
-	)
-	(no_connect
 		(at 127 46.99)
 	)
@@
 		)
 		(stroke
+			(width 0)
+			(type default)
+		)
+	)
+	(wire
+		(pts
+			(xy 74.93 72.39) (xy 92.71 72.39)
+		)
+		(stroke
